File: eps/eps.kicad_pcb (KiCad board)
At the start: 2 copper layers, 89.4 x 99.3 mm, 171 parts, among them J1 Screw_Panel, J10 Conn_Solar_3, J11 Conn_Solar_4, J12 Conn_I2C, J13 Conn_Star, J14 Conn_Wheel, J15 Conn_Deploy, J16 Conn_Comm, J17 Conn_Zone1, J18 Conn_Zone2, J2 Conn_Batt1, J21 Conn_Prop, J22 Conn_Pwr1, J23 Conn_Pwr2, J26 Conn_GPR, J27 Conn_Power, J3 Conn_Batt2, J4 Conn_Panel, J5 Conn_MPPT, J6 Conn_Balance, J7 Conn_Alerts, J8 Conn_Solar_1, J9 Conn_Solar_2, Q1 IRF7607PBF, Q10 CSD16403Q5A, Q11 CSD16403Q5A, Q2 IRF7607PBF, Q3 IRF7606PBF, Q4 IRF7606PBF, Q5 CSD16403Q5A, Q6 CSD16403Q5A, Q7 CSD16403Q5A, Q8 CSD16403Q5A, Q9 CSD16403Q5A, U1 AD5259BRMZ100, U10 TPS24701DGKR, U11 INA219BxD, U12 INA219BxD, U13 INA219BxD, U14 INA219BxD, U15 LM2936-3.3, U16 LM2936-3.3, U17 TPS24701DGKR, U18 TPS24701DGKR, U19 TPS24701DGKR, U2 LTC2943, U20 INA219BxD, U21 INA219BxD, U22 INA219BxD, U3 LT8611, U4 TCA9535DBR, U5 INA219BxD, U6 TCA9535DBR, U7 TPS24701DGKR, U8 TPS24701DGKR, U9 TPS24701DGKR

Commit message: Finalizing stuff
Replaced some out of stock parts, fixed some mistakes
Parts:
- removed Q1, Q2: IRF7607PBF, Package_SO:MSOP-8_3x3mm_P0.65mm
- removed Q3, Q4: IRF7606PBF, Package_SO:MSOP-8_3x3mm_P0.65mm
- added U23: AO6608, Package_TO_SOT_SMD:SOT-23-6_Handsoldering, F.Cu at (149.1, 37.3)
- added U24: AO6608, Package_TO_SOT_SMD:SOT-23-6_Handsoldering, F.Cu at (162.3, 39.8)
- C13, C14, C15, C16, C43, C44, C45: value 56n -> 68n
- C35, C37, C39, C40, C58, C59, C60: footprint Capacitor_THT:CP_Radial_D6.3mm_P2.50mm -> Capacitor_THT:CP_Radial_D8.0mm_P3.50mm
- R13: value 172k -> 150k
- R6, R7: footprint Resistor_SMD:R_0805_2012Metric_Pad1.20x1.40mm_HandSolder -> Resistor_SMD:R_2512_6332Metric_Pad1.40x3.35mm_HandSolder
- moved R3 17.5 mm to (145.5, 37.8), turned to 270 degrees
- moved R2 14.3 mm to (159.9, 36.7)
- moved R1 11.3 mm to (146.7, 34.3)
- moved R7 10.2 mm to (161.3, 44.3), turned to 0 degrees
- moved C31 8.18 mm to (114.6, 99.7), turned to 270 degrees
- moved R6 7.77 mm to (152.5, 41.3), turned to 0 degrees
- moved R4 7.00 mm to (158.6, 40.3)
- moved C35 3.07 mm to (108.8, 98.2), turned to 270 degrees
- moved C60 2.51 mm to (185.2, 101.6)
- moved C55 2.50 mm to (159.0, 110.7)
- moved C56 2.47 mm to (170.1, 110.7)
- moved C34 2.09 mm to (147.8, 110.7)
- moved C32 1.80 mm to (124.5, 110.7)
- moved C59 1.63 mm to (171.7, 105.2)
- moved J13 1.52 mm to (112.3, 115.1)
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Routing:
- net +BATT: track 352.3 -> 365.5 mm
- net Net-(R3-Pad2): track 19.0 -> 6.59 mm
- net BATT2: track 46.5 -> 55.8 mm
- net BAL1: track 16.4 -> 9.06 mm
- net OUT_POWER_SWITCH: track 131.9 -> 138.5 mm
- net GND: track 395.9 -> 401.6 mm, vias 73 -> 75
- net Net-(R4-Pad2): track 10.9 -> 6.90 mm
- net Net-(R7-Pad1): track 3.74 -> 6.96 mm
- net BATT1: track 36.9 -> 39.1 mm
- net Net-(C56-Pad1): track 27.8 -> 29.5 mm
- net Net-(D4-Pad1): track 9.57 -> 11.1 mm
- net Net-(C34-Pad1): track 28.8 -> 30.4 mm
- net Net-(C33-Pad1): track 28.2 -> 29.8 mm
- net Net-(C55-Pad1): track 27.9 -> 29.4 mm
- net Net-(Q5-Pad5): track 34.0 -> 35.1 mm
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