File: eps/eps.sch (KiCad schematic (older format))
At the start: 171 parts, among them J1 Screw_Panel, J10 Conn_Solar_3, J11 Conn_Solar_4, J12 Conn_I2C, J13 Conn_Star, J14 Conn_Wheel, J15 Conn_Deploy, J16 Conn_Comm, J17 Conn_Zone1, J18 Conn_Zone2, J2 Conn_Batt1, J21 Conn_Prop, J22 Conn_Pwr1, J23 Conn_Pwr2, J26 Conn_GPR, J27 Conn_Power, J3 Conn_Batt2, J4 Conn_Panel, J5 Conn_MPPT, J6 Conn_Balance, J7 Conn_Alerts, J8 Conn_Solar_1, J9 Conn_Solar_2, Q1 IRF7607PBF, Q10 CSD16403Q5A, Q11 CSD16403Q5A, Q2 IRF7607PBF, Q3 IRF7606PBF, Q4 IRF7606PBF, Q5 CSD16403Q5A, Q6 CSD16403Q5A, Q7 CSD16403Q5A, Q8 CSD16403Q5A, Q9 CSD16403Q5A, U1 AD5259BRMZ100, U10 TPS24701DGKR, U11 INA219BxD, U12 INA219BxD, U13 INA219BxD, U14 INA219BxD, U15 LM2936-3.3, U16 LM2936-3.3, U17 TPS24701DGKR, U18 TPS24701DGKR, U19 TPS24701DGKR, U2 LTC2943, U20 INA219BxD, U21 INA219BxD, U22 INA219BxD, U3 LT8611, U4 TCA9535DBR, U5 INA219BxD, U6 TCA9535DBR, U7 TPS24701DGKR, U8 TPS24701DGKR, U9 TPS24701DGKR

Commit message: Finalizing stuff
Replaced some out of stock parts, fixed some mistakes
Parts:
- removed Q1, Q2: IRF7607PBF, Package_SO:MSOP-8_3x3mm_P0.65mm, symbol Transistor_FET:IRF7607PBF
- removed Q3, Q4: IRF7606PBF, Package_SO:MSOP-8_3x3mm_P0.65mm, symbol Transistor_FET:IRF7606PBF
- added U23, U24: AO6608, Package_TO_SOT_SMD:SOT-23-6_Handsoldering, symbol eps-rescue:AO6608-HS2_Parts
- C1, C10, C11, C17, C18, C19, C20, C41, C42, C46, C47, C48: Part (none) -> C15850
- C12, C2, C22, C23, C24, C25, C27, C28, C29, C30, C31, C32, C33, C34, C36, C38, C49, C50, C51, C52, C53, C54, C55, C56, C57, C6: Part (none) -> C49678
- C13, C14, C15, C16, C43, C44, C45: value 56n -> 68n; Part (none) -> C1756
- C21, C4: Part (none) -> C1779
- C26, C5, R10: note (none) -> https://www.digikey.com/en/products/detail/panasonic-electr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
- C3, C7, C8: Part (none) -> C28323
- C35, C37, C39, C40, C58, C59, C60: footprint Capacitor_THT:CP_Radial_D6.3mm_P2.50mm -> Capacitor_THT:CP_Radial_D8.0mm_P3.50mm; note (none) -> https://www.digikey.com/en/products/detail/nichicon/UFW1C47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
- C9: Part (none) -> C1785
- D1, D2: Part (none) -> C2500
- D4, R18, R29, R30, R31, R32, R43, R44, R45: note (none) -> https://www.digikey.com/en/products/detail/rohm-semiconduct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
- H1, H2, H3, H4: Part (none) -> x; note (none) -> x
- J1: note (none) -> https://www.digikey.com/en/products/detail/phoenix-contact/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
- J10, J11, J12, J17, J18, J4, J5, J6, J7, J8, J9: note (none) -> https://www.digikey.com/en/products/detail/jst-sales-americ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
- J13, J14, J15, J16, J2, J21, J22, J23, J26, J27, J3: note (none) -> https://www.digikey.com/en/products/detail/molex/0430450212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
- L1: note (none) -> https://www.digikey.com/en/products/detail/chilisin-electro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
- Q10, Q11, Q5, Q6, Q7, Q8, Q9, U11, U12, U13, U14, U15, U16, U20, U21, U22, U4, U5, U6: note (none) -> https://www.digikey.com/en/products/detail/texas-instrument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
- R1, R17, R19, R2, R20, R21, R22, R23, R24, R25, R26, R3, R37, R38, R39, R4, R40, R41, R42, R8: Part (none) -> C17414
- R12, R15: note (none) -> https://www.digikey.com/en/products/detail/delta-electronic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
- R13: value 172k -> 150k; Part (none) -> C17470
- R14: Part (none) -> C17514
- R16, R27, R28: Part (none) -> C26010
- R33, R34, R35, R36, R46, R47, R48: Part (none) -> C17415
- R5: Part (none) -> C17767
- R6, R7: footprint Resistor_SMD:R_0805_2012Metric_Pad1.20x1.40mm_HandSolder -> Resistor_SMD:R_2512_6332Metric_Pad1.40x3.35mm_HandSolder; note (none) -> https://www.digikey.com/en/products/detail/stackpole-electr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
- R9: note (none) -> https://www.digikey.com/en/products/detail/koa-speer-electr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
- U1: symbol HS2_Parts:AD5259BRMZ100 -> eps-rescue:AD5259BRMZ100-HS2_Parts; note (none) -> https://www.digikey.com/en/products/detail/analog-devices-i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
- U10, U17, U18, U19, U7, U8, U9: symbol HS2_Parts:TPS24701DGKR -> eps-rescue:TPS24701DGKR-HS2_Parts; note (none) -> https://www.digikey.com/en/products/detail/texas-instrument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
- U2: symbol HS2_Parts:LTC2943 -> eps-rescue:LTC2943-HS2_Parts; note (none) -> https://www.digikey.com/en/products/detail/LTC2943CDD%23PBF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
- U3: symbol HS2_Parts:LT8611 -> eps-rescue:LT8611-HS2_Parts; note (none) -> https://www.digikey.com/en/products/detail/analog-devices-i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
Connections:
- net BAL1: now also U23.1 (G1)
- net BAL2: now also U24.1 (G1)
- net BATT1: now also U24.2 (S2)
- net BATT2: now also U23.2 (S2)
- net GND: now also U23.5 (S1), U24.5 (S1)
- net at R3.2: now also U23.3 (G2), U23.6 (D1)
- net at R6.1: now also U23.4 (D2)
- net at R4.2: now also U24.3 (G2), U24.6 (D1)
- net at R7.1: now also U24.4 (D2)
Other:
- moved on the sheet: R1, R2, R3, R4, R6, R7
