File: testing boards/BQ298xyz/BQ298xyz.sch (KiCad schematic (older format))
At the start: 9 parts, among them J1 XT30, U1 1048-2S-18650-Holder, U2 BQ298xyz

Commit message: Did work
Finished a board, maybe forgot to commit some a while ago?
Parts:
- gave numbers to parts that had none: 1
Changed lines of the file:
@@
 	8250 4600 8500 4600
 $Comp
-L HS2_Parts:EFC2K103NUZTDG U?
+L HS2_Parts:EFC2K103NUZTDG U3
 U 1 1 61B5E55D
 P 5800 3650
-F 0 "U?" H 6744 3696 50  0000 L CNN
+F 0 "U3" H 6744 3696 50  0000 L CNN
 F 1 "EFC2K103NUZTDG" H 6744 3605 50  0000 L CNN
 F 2 "HS2_parts:EFC2K103NUZTDG" H 6300 3450 50  0001 C CNN
