File: testing boards/INA219/INA219_Breakout/INA219_Breakout.kicad_pcb (KiCad board)
At the start: 2 copper layers, 10.2 x 20.3 mm, 7 parts, among them J1 Conn_01x04_Male, J2 Conn_01x04_Male, U1 INA219B

Commit message: Did work
Finished a board, maybe forgot to commit some a while ago?
Other:
- net class Default removed
