File: testing boards/TPS2595x1_Breakout/TPS2595x1_Breakout.kicad_pcb (KiCad board)
At the start: 2 copper layers, 8.3 x 10.2 mm, 9 parts, among them J1 Pin Header, U1 TPS2595x1

Commit message: Did work
Finished a board, maybe forgot to commit some a while ago?
Other:
- board size 8.3 x 10.2 mm -> 10.2 x 10.2 mm
- board text added: "FLT"
- board text added: "G"
- board text added: "IN"
- board text added: "OUT"
Changed lines of the file:
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@@
   (general
     (thickness 1.6)
-    (drawings 4)
+    (drawings 12)
     (tracks 42)
     (zones 0)
@@
     (38 B.Mask user)
     (39 F.Mask user)
-    (40 Dwgs.User user)
+    (40 Dwgs.User user hide)
     (41 Cmts.User user)
     (42 Eco1.User user)
@@
     (46 B.CrtYd user hide)
     (47 F.CrtYd user hide)
-    (48 B.Fab user)
+    (48 B.Fab user hide)
     (49 F.Fab user hide)
   )
@@
     (pcbplotparams
       (layerselection 0x010fc_ffffffff)
-      (usegerberextensions false)
-      (usegerberattributes true)
-      (usegerberadvancedattributes true)
-      (creategerberjobfile true)
+      (usegerberextensions true)
+      (usegerberattributes false)
+      (usegerberadvancedattributes false)
+      (creategerberjobfile false)
       (excludeedgelayer true)
       (linewidth 0.100000)
@@
       (psa4output false)
       (plotreference true)
-      (plotvalue true)
+      (plotvalue false)
       (plotinvisibletext false)
       (padsonsilk false)
-      (subtractmaskfromsilk false)
+      (subtractmaskfromsilk true)
       (outputformat 1)
       (mirror false)
-      (drillshape 1)
+      (drillshape 0)
       (scaleselection 1)
-      (outputdirectory ""))
+      (outputdirectory "tps2595x1_gerber/"))
   )
   (net 0 "")
@@
     )
   )
-  (gr_line (start 133.35 114.3) (end 133.35 104.14) (layer Edge.Cuts) (width 0.05))
-  (gr_line (start 141.605 114.3) (end 133.35 114.3) (layer Edge.Cuts) (width 0.05))
-  (gr_line (start 141.605 104.14) (end 141.605 114.3) (layer Edge.Cuts) (width 0.05))
-  (gr_line (start 133.35 104.14) (end 141.605 104.14) (layer Edge.Cuts) (width 0.05))
+  (gr_text G (at 132.4 113.03) (layer F.SilkS)
+    (effects (font (size 1 1) (thickness 0.15)))
+  )
+  (gr_text FLT (at 132.4 110.9 90) (layer F.SilkS)
+    (effects (font (size 1 1) (thickness 0.15)))
+  )
+  (gr_text OUT (at 132.4 108.1 90) (layer F.SilkS)
+    (effects (font (size 1 1) (thickness 0.15)))
+  )
+  (gr_text IN (at 132.5 105.6 90) (layer F.SilkS)
+    (effects (font (size 1 1) (thickness 0.15)))
+  )
+  (gr_line (start 131.445 106.045) (end 131.445 112.395) (layer Edge.Cuts) (width 0.05))
+  (gr_arc (start 139.7 106.045) (end 141.605 106.045) (angle -90) (layer Edge.Cuts) (width 0.05))
+  (gr_arc (start 139.7 112.395) (end 139.7 114.3) (angle -90) (layer Edge.Cuts) (width 0.05))
+  (gr_arc (start 133.35 112.395) (end 131.445 112.395) (angle -90) (layer Edge.Cuts) (width 0.05))
+  (gr_arc (start 133.35 106.045) (end 133.35 104.14) (angle -90) (layer Edge.Cuts) (width 0.05))
+  (gr_line (start 139.7 114.3) (end 133.35 114.3) (layer Edge.Cuts) (width 0.05))
+  (gr_line (start 141.605 106.045) (end 141.605 112.395) (layer Edge.Cuts) (width 0.05))
+  (gr_line (start 133.35 104.14) (end 139.7 104.14) (layer Edge.Cuts) (width 0.05))
   (via (at 137.16 113.03) (size 0.8) (drill 0.4) (layers F.Cu B.Cu) (net 1))
   (via (at 139.7 113.03) (size 0.8) (drill 0.4) (layers F.Cu B.Cu) (net 1))
